Commit message: Alterando o arquivo para usar a camera como um macro

File: Simulação/Martha_ws/src/martha_description/urdf/camera.xacro (robot description, xacro)
@@ -1,27 +1,46 @@
-<?xml version="1.0" ?>
+<?xml version="1.0"?>
 <robot xmlns:xacro="http://www.ros.org/wiki/xacro">
-    <xacro:property name="body_color" value="Gazebo/Silver" />
-    <gazebo reference="cabeca_1">
-        <material>Gazebo/Silver</material>
-        <sensor name="camera" type="camera">
-            <pose> -0.02060 -0.050864 0.047202 0 0 -1.57 </pose>
-            <visualize>true</visualize>
-            <update_rate>10</update_rate>
-            <camera>
-                <horizontal_fov>1.089</horizontal_fov>
+    <xacro:macro name="camera_sensor" params="parent camera_name ns origin">
+        <!-- camera -->
+        <gazebo reference="${parent}">
+            <sensor type="camera" name="${camera_name}">
+            <pose>${origin}</pose>
+            <update_rate>30.0</update_rate>
+            <camera name="head">
+                <horizontal_fov>1.3962634</horizontal_fov>
                 <image>
-                    <format>R8G8B8</format>
-                    <width>640</width>
-                    <height>480</height>
+                <width>640</width>
+                <height>480</height>
+                <format>R8G8B8</format>
                 </image>
                 <clip>
-                    <near>0.05</near>
-                    <far>8.0</far>
+                <near>0.02</near>
+                <far>300</far>
                 </clip>
+                <noise>
+                <type>gaussian</type>
+                <!-- Noise is sampled independently per pixel on each frame.
+                    That pixel's noise value is added to each of its color
+                    channels, which at that point lie in the range [0,1]. -->
+                <mean>0.0</mean>
+                <stddev>0.007</stddev>
+                </noise>
             </camera>
             <plugin name="camera_controller" filename="libgazebo_ros_camera.so">
-                <frame_name>cabeca_1</frame_name>
+                <alwaysOn>true</alwaysOn>
+                <updateRate>0.0</updateRate>
+                <cameraName>/${ns}/${camera_name}</cameraName>
+                <imageTopicName>image_raw</imageTopicName>
+                <cameraInfoTopicName>camera_info</cameraInfoTopicName>
+                <frameName>${parent}</frameName>
+                <hackBaseline>0.07</hackBaseline>
+                <distortionK1>0.0</distortionK1>
+                <distortionK2>0.0</distortionK2>
+                <distortionK3>0.0</distortionK3>
+                <distortionT1>0.0</distortionT1>
+                <distortionT2>0.0</distortionT2>
             </plugin>
-        </sensor>
-    </gazebo>
+            </sensor>
+        </gazebo>
+    </xacro:macro>
 </robot>
